File: TechStarter.kicad_pcb (KiCad board)
At the start: 4 copper layers, 100 x 112.5 mm, 83 parts, among them J1 Conn_01x04_Socket, J10 Conn_01x03_Socket, J11 Conn_01x03_Socket, J12 Conn_01x04_Pin, J13 Conn_01x02_Socket, J14 Conn_01x04_Socket, J15 Conn_01x04_Socket, J16 Conn_01x02_Socket, J17 Conn_01x02_Socket, J18 Conn_01x04_Socket, J2 Conn_01x04_Socket, J3 Conn_01x02_Socket, J4 Conn_01x04_Socket, J5 Conn_01x03_Socket, J6 Conn_01x04_Socket, J7 Conn_01x03_Socket, J8 Conn_01x03_Socket, J9 Conn_01x03_Socket, Q3 IRLZ44N, U1 STM32F446RETx, U10 PC817, U11 AMS1117-3.3, U12 TP4056-42-ESOP8, U2 TMC2209-LA, U3 TMC2209-LA, U4 LM2596S-3.3, U5 MX25L3233FM1, U6 TMC2209-LA, U7 AMS1117-3.3, U8 TMC2209-LA, U9 PC817

Commit message: ,
,
Parts:
- added FID1: Fiducial, Fiducial:Fiducial_0.75mm_Mask1.5mm, F.Cu at (212.2, 50.0)
- added FID2: Fiducial, Fiducial:Fiducial_0.75mm_Mask1.5mm, F.Cu at (205.5, 93.0)
- added FID3: Fiducial, Fiducial:Fiducial_0.75mm_Mask1.5mm, F.Cu at (205.2, 109.8)
- added FID4: Fiducial, Fiducial:Fiducial_0.75mm_Mask1.5mm, F.Cu at (240.5, 80.5)
- added FID5: Fiducial, Fiducial:Fiducial_0.75mm_Mask1.5mm, F.Cu at (252.5, 104.8)
- added FID6: Fiducial, Fiducial:Fiducial_0.75mm_Mask1.5mm, F.Cu at (206.5, 118.2)
- added FID7: Fiducial, Fiducial:Fiducial_0.75mm_Mask1.5mm, F.Cu at (235.0, 93.5)
- added FID8: Fiducial, Fiducial:Fiducial_0.75mm_Mask1.5mm, F.Cu at (220.5, 75.2)
Routing:
- net GND: vias 851 -> 831
Other:
- outline, holes or cut-outs redrawn

Commit message: Resistor update
Nigger
Parts:
- R11: value 220R -> 120R
- R20: value 2,7k -> 1,2k

Commit message: resist
zase jsem změnil hodnotu rezistorů :)
Parts:
- R11: value 120R -> 220R
- R20: value 1,2k -> 2,4k
Changed lines of the file:
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@@
 			)
 		)
-		(property "Value" "120R"
+		(property "Value" "220R"
 			(at 0 1.43 90)
 			(layer "F.Fab")
@@
 			)
 		)
-		(property "Value" "1,2k"
+		(property "Value" "2,4k"
 			(at 0 1.43 0)
 			(layer "F.Fab")
