File: TechStarter.kicad_pcb (KiCad board)
At the start: 4 copper layers, 100 x 112.5 mm, 91 parts, among them J1 Conn_01x04_Socket, J10 Conn_01x03_Socket, J11 Conn_01x03_Socket, J12 Conn_01x04_Pin, J13 Conn_01x02_Socket, J14 Conn_01x04_Socket, J15 Conn_01x04_Socket, J16 Conn_01x02_Socket, J17 Conn_01x02_Socket, J18 Conn_01x04_Socket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

Commit message: 3D models
Parts:
- U12: footprint Package_SO:SOIC-8-1EP_3.9x4.9mm_P1.27mm_EP2.41x3.3mm_ThermalVias -> Package_SO:SOIC-8-1EP_3.9x4.9mm_P1.27mm_EP2.41x3.3mm_ThermalVias_model
