File: Logic block.kicad_sch (KiCad schematic)
At the start: 44 parts, among them J1 Conn_01x04_Socket, J14 Conn_01x04_Socket, J15 Conn_01x04_Socket, J16 Conn_01x02_Socket, J18 Conn_01x04_Socket, J2 Conn_01x04_Socket, J3 Conn_01x02_Socket, J4 Conn_01x04_Socket, J6 Conn_01x04_Socket, Q3 IRLZ44N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

Commit message: Resistor Value
 i found that you are an idiot sandwich
Parts:
- R11: value 220R -> 120R
- R20: value 2,7k -> 1,2k
