File: powerbrick.kicad_sch (KiCad schematic)
At the start: 20 parts, among them J13 Conn_01x02_Socket, J17 Conn_01x02_Socket, U11 AMS1117-3.3, U12 TP4056-42-ESOP8, U4 LM2596S-3.3, U7 AMS1117-3.3

Commit message: 3D models
Parts:
- U12: footprint Package_SO:SOIC-8-1EP_3.9x4.9mm_P1.27mm_EP2.41x3.3mm_ThermalVias -> Package_SO:SOIC-8-1EP_3.9x4.9mm_P1.27mm_EP2.41x3.3mm_ThermalVias_model
Changed lines of the file:
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@@
 			)
 		)
-		(property "Footprint" "Package_SO:SOIC-8-1EP_3.9x4.9mm_P1.27mm_EP2.41x3.3mm_ThermalVias"
+		(property "Footprint" "Package_SO:SOIC-8-1EP_3.9x4.9mm_P1.27mm_EP2.41x3.3mm_ThermalVias_model"
 			(at 140.208 106.68 0)
 			(effects
